File: kicad-project/capstone.kicad_sch (KiCad schematic)
At the start: 0 parts

Commit message: various things (forgot to commit)
Other:
- added sheet Address Register (addr.kicad_sch)
- sheet RAM ports: added RE, WE, Word Select; removed none
- sheet ROM ports: added none; removed Address

Commit message: address register and more
Other:
- sheet Address Register ports: added Bus, RAM, ROM; removed none
- sheet ROM ports: added Address; removed none
Changed lines of the file:
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@@
 (kicad_sch (version 20211123) (generator eeschema)
   (paper "A4")
+  (junction (at 133.35 76.2) (diameter 0) (color 0 0 0 0)
+  )
   (junction (at 133.35 107.95) (diameter 0) (color 0 0 0 0)
   )
@@
     (stroke (width 0) (type default) (color 0 0 0 0))
   )
-  (bus (pts (xy 133.35 57.15) (xy 133.35 82.55))
+  (bus (pts (xy 133.35 57.15) (xy 133.35 76.2))
     (stroke (width 0) (type default) (color 0 0 0 0))
   )
@@
     (stroke (width 0) (type default) (color 0 0 0 0))
   )
+  (bus (pts (xy 114.3 76.2) (xy 133.35 76.2))
+    (stroke (width 0) (type default) (color 0 0 0 0))
+  )
   (bus (pts (xy 182.88 63.5) (xy 182.88 76.2))
     (stroke (width 0) (type default) (color 0 0 0 0))
@@
     (stroke (width 0) (type default) (color 0 0 0 0))
   )
+  (bus (pts (xy 133.35 76.2) (xy 133.35 82.55))
+    (stroke (width 0) (type default) (color 0 0 0 0))
+  )
   (bus (pts (xy 182.88 38.1) (xy 182.88 44.45))
     (stroke (width 0) (type default) (color 0 0 0 0))
@@
     (stroke (width 0) (type default) (color 0 0 0 0))
   )
+  (bus (pts (xy 85.09 82.55) (xy 85.09 88.9))
+    (stroke (width 0) (type default) (color 0 0 0 0))
+  )
   (bus (pts (xy 68.58 101.6) (xy 68.58 114.3))
     (stroke (width 0) (type default) (color 0 0 0 0))
   )
+  (label "b0-b3" (at 114.3 120.65 0)
+    (effects (font (size 1.27 1.27)) (justify left bottom))
+  )
+  (label "0-3" (at 68.58 107.95 0)
+    (effects (font (size 1.27 1.27)) (justify left bottom))
+  )
+  (label "b0-b3" (at 148.59 82.55 180)
+    (effects (font (size 1.27 1.27)) (justify right bottom))
+  )
+  (label "0-3" (at 73.66 133.35 0)
+    (effects (font (size 1.27 1.27)) (justify left bottom))
+  )
+  (label "b0-b3" (at 148.59 31.75 180)
+    (effects (font (size 1.27 1.27)) (justify right bottom))
+  )
+  (label "b0-b3" (at 114.3 57.15 0)
+    (effects (font (size 1.27 1.27)) (justify left bottom))
+  )
+  (label "a0-a7" (at 85.09 86.36 0)
+    (effects (font (size 1.27 1.27)) (justify left bottom))
+  )
+  (label "b0-b3" (at 152.4 107.95 180)
+    (effects (font (size 1.27 1.27)) (justify right bottom))
+  )
+  (label "b0-b3" (at 114.3 76.2 0)
+    (effects (font (size 1.27 1.27)) (justify left bottom))
+  )
+  (label "b0-b3" (at 114.3 31.75 0)
+    (effects (font (size 1.27 1.27)) (justify left bottom))
+  )
   (sheet (at 152.4 101.6) (size 63.5 12.7) (fields_autoplaced)
     (stroke (width 0.1524) (type solid) (color 0 0 0 0))
@@
       (effects (font (size 1.27 1.27)) (justify left top))
     )
+    (pin "Bus" input (at 114.3 76.2 0)
+      (effects (font (size 1.27 1.27)) (justify right))
+    )
+    (pin "ROM" output (at 85.09 82.55 270)
+      (effects (font (size 1.27 1.27)) (justify left))
+    )
+    (pin "RAM" output (at 85.09 69.85 90)
+      (effects (font (size 1.27 1.27)) (justify right))
+    )
   )
   (sheet (at 228.6 25.4) (size 20.32 13.97) (fields_autoplaced)
@@
       (effects (font (size 1.27 1.27)) (justify left))
     )
+    (pin "Address" input (at 85.09 88.9 90)
+      (effects (font (size 1.27 1.27)) (justify right))
+    )
   )
   (sheet (at 152.4 25.4) (size 63.5 12.7) (fields_autoplaced)
@@
       (effects (font (size 1.27 1.27)) (justify right))
     )
-    (pin "Out" input (at 68.58 127 270)
+    (pin "Out" output (at 68.58 127 270)
       (effects (font (size 1.27 1.27)) (justify left))
     )
@@
       (reference "#PWR0101") (unit 1) (value "GND") (footprint "")
     )
-    (path "/6a99f3bb-c052-48d8-9231-331d6493db5e/9339b645-b42c-41f5-bb54-ffed7e58eaba"
-      (reference "#PWR0102") (unit 1) (value "+5V") (footprint "")
-    )
-    (path "/6a99f3bb-c052-48d8-9231-331d6493db5e/e2c4cd5c-1ad0-4913-ba91-d37149301ef1"
-      (reference "#PWR0103") (unit 1) (value "+5V") (footprint "")
-    )
     (path "/6a99f3bb-c052-48d8-9231-331d6493db5e/3f45ef44-f5bd-4af3-938f-f34da65c4756"
       (reference "#PWR0104") (unit 1) (value "GND") (footprint "")
     )
-    (path "/6a99f3bb-c052-48d8-9231-331d6493db5e/e32109fe-5a57-4270-b31f-3afb5d146347"
-      (reference "#PWR0105") (unit 1) (value "+5V") (footprint "")
-    )
     (path "/6a99f3bb-c052-48d8-9231-331d6493db5e/86742743-bfb9-4581-99da-04aaf2734226"
       (reference "#PWR0106") (unit 1) (value "GND") (footprint "")
     )
-    (path "/6a99f3bb-c052-48d8-9231-331d6493db5e/4f2aaaab-8e64-440a-8589-8dfdaf1a1c22"
-      (reference "#PWR0107") (unit 1) (value "+5V") (footprint "")
-    )
     (path "/6a99f3bb-c052-48d8-9231-331d6493db5e/734e7094-42b6-4749-aa48-38b0cadfd576"
       (reference "#PWR0108") (unit 1) (value "GND") (footprint "")
@@
       (reference "#PWR0109") (unit 1) (value "GND") (footprint "")
     )
-    (path "/6a99f3bb-c052-48d8-9231-331d6493db5e/a4a75b4b-53a5-4a8d-a1d8-a1fa90dd9d1a"
-      (reference "#PWR0110") (unit 1) (value "+5V") (footprint "")
-    )
     (path "/43d661c2-7442-45d8-9a0c-31aec2786e4e/970475e0-e139-4ee8-bb57-6f83d31a7ac7"
       (reference "#PWR0111") (unit 1) (value "+5V") (footprint "")
@@
       (reference "#PWR0114") (unit 1) (value "GND") (footprint "")
     )
+    (path "/6a99f3bb-c052-48d8-9231-331d6493db5e/143663e9-5ded-487a-bfcd-944ee09c84a6"
+      (reference "#PWR?") (unit 1) (value "VCC") (footprint "")
+    )
+    (path "/40298a9c-5a74-4acd-aa00-c14644bf8e5a/2d06b0b0-0a43-4b6e-8f53-32d230a77661"
+      (reference "#PWR?") (unit 1) (value "VCC") (footprint "")
+    )
+    (path "/40298a9c-5a74-4acd-aa00-c14644bf8e5a/2e88e62e-f8b6-4c3b-bc84-9640478b5b58"
+      (reference "#PWR?") (unit 1) (value "GND") (footprint "")
+    )
+    (path "/40298a9c-5a74-4acd-aa00-c14644bf8e5a/9e3d9fd2-2db2-43c6-8a47-722997e8f865"
+      (reference "#PWR?") (unit 1) (value "GND") (footprint "")
+    )
+    (path "/6a99f3bb-c052-48d8-9231-331d6493db5e/a6905929-b7f9-4812-a6b6-9a0605d2d2eb"
+      (reference "#PWR?") (unit 1) (value "VCC") (footprint "")
+    )
+    (path "/40298a9c-5a74-4acd-aa00-c14644bf8e5a/b72702d3-179f-4f8b-a086-21d6564cebc8"
+      (reference "#PWR?") (unit 1) (value "VCC") (footprint "")
+    )
+    (path "/40298a9c-5a74-4acd-aa00-c14644bf8e5a/cd16440a-88e7-4b15-ae79-a464d2e787b3"
+      (reference "#PWR?") (unit 1) (value "GND") (footprint "")
+    )
+    (path "/6a99f3bb-c052-48d8-9231-331d6493db5e/d4b193a5-b397-4f8b-97d9-141c57f782b5"
+      (reference "#PWR?") (unit 1) (value "VCC") (footprint "")
+    )
+    (path "/6a99f3bb-c052-48d8-9231-331d6493db5e/deece549-762e-47fa-a3af-e336749e4d78"
+      (reference "#PWR?") (unit 1) (value "VCC") (footprint "")
+    )
+    (path "/6a99f3bb-c052-48d8-9231-331d6493db5e/eb6474fe-a81f-4a46-98ca-174ac8d8673e"
+      (reference "#PWR?") (unit 1) (value "VCC") (footprint "")
+    )
     (path "/43d661c2-7442-45d8-9a0c-31aec2786e4e/7590cf82-bd59-405b-a431-798e6366d885"
       (reference "C1") (unit 1) (value "CAP") (footprint "")
@@
       (reference "U5") (unit 1) (value "LM555xN") (footprint "Package_DIP:DIP-8_W7.62mm")
     )
-  )
+    (path "/40298a9c-5a74-4acd-aa00-c14644bf8e5a/33b56775-6531-4769-a629-5b2630ad4d20"
+      (reference "U?") (unit 1) (value "74LS173") (footprint "")
+    )
+    (path "/40298a9c-5a74-4acd-aa00-c14644bf8e5a/c1ff06ab-76bc-4192-a411-d87ee2c796cd"
+      (reference "U?") (unit 1) (value "74LS173") (footprint "")
+    )
+  )
